File: pcb/Eule.kicad_pcb (KiCad board)
At the start: 2 copper layers, 50 x 76.5 mm, 8 parts, among them J1 Conn_01x03_Male

Commit message: v2.0
changed switch
increased footprint for batterie holder
text
Parts:
- removed J1: Conn_01x03_Male, Connector_Harwin:Harwin_M20-89003xx_1x03_P2.54mm_Horizontal
- added SW1: SW_DPDT_x2, MSS22D18G2:MSS22D18G2, B.Cu at (56.0, 88.0)
Routing:
- net Net-(BT1-Pad2): track 29.9 -> 25.1 mm
Other:
- board text added: "Obnoxious Owl"
- board text added: "Unausstehlich Eule"

Commit message: footprint enlarged Text changes LED arrow
Other:
- board text added: "Entnervte Eule"
- board text removed: "Unausstehlich Eule"
Changed lines of the file:
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@@
       (drillshape 0)
       (scaleselection 1)
-      (outputdirectory "Gerber/v1.0")
+      (outputdirectory "Gerber/v3.0")
     )
   )
@@
     (property "Sheetname" "")
     (attr smd)
-    (fp_text reference "SW1" (at 0.06 5 unlocked) (layer "B.SilkS")
+    (fp_text reference "SW1" (at 0 7.62 unlocked) (layer "B.SilkS")
       (effects (font (size 1 1) (thickness 0.15)) (justify mirror))
     )
-    (fp_text value "SW_DPDT_x2" (at 0 -5 unlocked) (layer "B.Fab")
+    (fp_text value "SW_DPDT_x2" (at 0 6.12 unlocked) (layer "B.Fab")
       (effects (font (size 1 1) (thickness 0.15)) (justify mirror))
     )
@@
     )
     (fp_rect (start -4.6 1.75) (end 4.6 -1.75) (layer "B.SilkS") (width 0.12) (fill none))
-    (pad "1" smd rect (at -2.5 2.95 90) (size 1.7 1.2) (layers "B.Cu" "B.Paste" "B.Mask")
+    (pad "1" smd rect (at -2.5 3.45 90) (size 2.7 1.2) (layers "B.Cu" "B.Paste" "B.Mask")
       (net 3 "GND") (pinfunction "A") (pintype "passive"))
-    (pad "2" smd rect (at 0 2.95 90) (size 1.7 1.2) (layers "B.Cu" "B.Paste" "B.Mask")
+    (pad "2" smd rect (at 0 3.45 90) (size 2.7 1.2) (layers "B.Cu" "B.Paste" "B.Mask")
       (net 2 "Net-(BT1-Pad2)") (pinfunction "B") (pintype "passive"))
-    (pad "3" smd rect (at 2.5 2.95 90) (size 1.7 1.2) (layers "B.Cu" "B.Paste" "B.Mask")
+    (pad "3" smd rect (at 2.5 3.45 90) (size 2.7 1.2) (layers "B.Cu" "B.Paste" "B.Mask")
       (net 6 "unconnected-(SW1-Pad3)") (pinfunction "C") (pintype "passive+no_connect"))
-    (pad "4" smd rect (at -2.5 -2.95 90) (size 1.7 1.2) (layers "B.Cu" "B.Paste" "B.Mask")
+    (pad "4" smd rect (at -2.5 -3.45 90) (size 2.7 1.2) (layers "B.Cu" "B.Paste" "B.Mask")
       (net 7 "unconnected-(SW1-Pad4)") (pinfunction "A") (pintype "passive+no_connect"))
-    (pad "5" smd rect (at 0 -2.95 90) (size 1.7 1.2) (layers "B.Cu" "B.Paste" "B.Mask")
+    (pad "5" smd rect (at 0 -3.45 90) (size 2.7 1.2) (layers "B.Cu" "B.Paste" "B.Mask")
       (net 8 "unconnected-(SW1-Pad5)") (pinfunction "B") (pintype "passive+no_connect"))
-    (pad "6" smd rect (at 2.5 -2.95 90) (size 1.7 1.2) (layers "B.Cu" "B.Paste" "B.Mask")
+    (pad "6" smd rect (at 2.5 -3.45 90) (size 2.7 1.2) (layers "B.Cu" "B.Paste" "B.Mask")
       (net 9 "unconnected-(SW1-Pad6)") (pinfunction "C") (pintype "passive+no_connect"))
   )
@@
       (xy 48.641 46.482)
     ) (layer "B.Mask") (width 0.15) (fill solid))
+  (gr_poly
+    (pts
+      (xy 61.6 50)
+      (xy 60.6 51)
+      (xy 60.1 49.5)
+    ) (layer "B.Mask") (width 0.2) (fill solid))
   (gr_circle (center 46.77 39.45) (end 51.77 39.45) (layer "B.Mask") (width 0.15) (fill solid))
   (gr_rect (start 46.77 34.45) (end 64.77 44.45) (layer "B.Mask") (width 0.15) (fill solid))
+  (gr_poly
+    (pts
+      (xy 50.9 50.9)
+      (xy 49.9 49.9)
+      (xy 51.4 49.4)
+    ) (layer "B.Mask") (width 0.2) (fill solid))
   (gr_circle (center 64.77 39.45) (end 69.77 39.45) (layer "B.Mask") (width 0.15) (fill solid))
   (gr_poly
@@
     (effects (font (size 1 1) (thickness 0.15)) (justify mirror))
   )
-  (gr_text "Unausstehlich Eule" (at 67 91 56) (layer "B.Mask")
+  (gr_text "Entnervte Eule" (at 67 91 56) (layer "B.Mask")
     (effects (font (size 1 1) (thickness 0.15)) (justify mirror))
   )
