File: pcb/Eule.kicad_sch (KiCad schematic)
At the start: 6 parts, among them J1 Conn_01x03_Male

Commit message: v2.0
changed switch
increased footprint for batterie holder
text
Parts:
- removed J1: Conn_01x03_Male, Connector_Harwin:Harwin_M20-89003xx_1x03_P2.54mm_Horizontal, symbol Connector:Conn_01x03_Male
- added SW1: SW_DPDT_x2, MSS22D18G2:MSS22D18G2, symbol Switch:SW_DPDT_x2
Connections:
- net GND: now also SW1.1 (A)
- net at BT1.2 (-): now also SW1.2 (B)
- no-connect marks 1 -> 4
Changed lines of the file:
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@@
   (title_block
     (title "Eule")
-    (date "2023-01-13")
-    (rev "v1.0")
+    (date "2023-02-02")
+    (rev "v2.0")
     (company "Kaulquappe(ZTL)")
   )
@@
   (junction (at 52.07 66.04) (diameter 0) (color 0 0 0 0)
   )
-  (no_connect (at 44.45 68.58))
+  (no_connect (at 38.1 82.55))
+  (no_connect (at 48.26 80.01))
+  (no_connect (at 48.26 71.12))
+  (no_connect (at 48.26 85.09))
   (wire (pts (xy 52.07 53.34) (xy 52.07 55.88))
     (stroke (width 0) (type default) (color 0 0 0 0))
   )
-  (wire (pts (xy 41.91 68.58) (xy 41.91 66.04))
-    (stroke (width 0) (type default) (color 0 0 0 0))
-  )
-  (wire (pts (xy 41.91 66.04) (xy 52.07 66.04))
+  (wire (pts (xy 33.02 60.96) (xy 33.02 68.58))
     (stroke (width 0) (type default) (color 0 0 0 0))
   )
@@
     (stroke (width 0) (type default) (color 0 0 0 0))
   )
-  (wire (pts (xy 39.37 66.04) (xy 39.37 68.58))
-    (stroke (width 0) (type default) (color 0 0 0 0))
-  )
-  (wire (pts (xy 33.02 66.04) (xy 39.37 66.04))
+  (wire (pts (xy 33.02 68.58) (xy 38.1 68.58))
+    (stroke (width 0) (type default) (color 0 0 0 0))
+  )
+  (wire (pts (xy 48.26 66.04) (xy 52.07 66.04))
     (stroke (width 0) (type default) (color 0 0 0 0))
   )
@@
     (stroke (width 0) (type default) (color 0 0 0 0))
   )
-  (wire (pts (xy 33.02 60.96) (xy 33.02 66.04))
-    (stroke (width 0) (type default) (color 0 0 0 0))
-  )
   (wire (pts (xy 33.02 57.15) (xy 33.02 60.96))
     (stroke (width 0) (type default) (color 0 0 0 0))
@@
     (stroke (width 0) (type default) (color 0 0 0 0))
   )
+  (symbol (lib_id "Switch:SW_DPDT_x2") (at 43.18 68.58 0) (unit 1)
+    (in_bom yes) (on_board yes) (fields_autoplaced)
+    (property "Reference" "SW1" (id 0) (at 43.18 60.96 0))
+    (property "Value" "SW_DPDT_x2" (id 1) (at 43.18 63.5 0))
+    (property "Footprint" "MSS22D18G2:MSS22D18G2" (id 2) (at 43.18 68.58 0)
+      (effects (font (size 1.27 1.27)) hide)
+    )
+    (property "Datasheet" "~" (id 3) (at 43.18 68.58 0)
+      (effects (font (size 1.27 1.27)) hide)
+    )
+    (pin "1")
+    (pin "2")
+    (pin "3")
+    (pin "4")
+    (pin "5")
+    (pin "6")
+  )
   (symbol (lib_id "Device:R") (at 52.07 49.53 0) (unit 1)
     (in_bom yes) (on_board yes) (fields_autoplaced)
@@
     (pin "1")
     (pin "2")
+  )
+  (symbol (lib_id "Switch:SW_DPDT_x2") (at 43.18 82.55 0) (unit 2)
+    (in_bom yes) (on_board yes) (fields_autoplaced)
+    (property "Reference" "SW1" (id 0) (at 43.18 74.93 0))
+    (property "Value" "SW_DPDT_x2" (id 1) (at 43.18 77.47 0))
+    (property "Footprint" "MSS22D18G2:MSS22D18G2" (id 2) (at 43.18 82.55 0)
+      (effects (font (size 1.27 1.27)) hide)
+    )
+    (property "Datasheet" "~" (id 3) (at 43.18 82.55 0)
+      (effects (font (size 1.27 1.27)) hide)
+    )
+    (pin "1")
+    (pin "2")
+    (pin "3")
+    (pin "4")
+    (pin "5")
+    (pin "6")
   )
   (symbol (lib_id "power:PWR_FLAG") (at 31.75 60.96 90) (unit 1)
@@
     )
     (pin "1")
-  )
-  (symbol (lib_id "Connector:Conn_01x03_Male") (at 41.91 73.66 90) (unit 1)
-    (in_bom yes) (on_board yes) (fields_autoplaced)
-    (property "Reference" "J1" (id 0) (at 41.91 76.2 90))
-    (property "Value" "Conn_01x03_Male" (id 1) (at 41.91 78.74 90))
-    (property "Footprint" "Connector_Harwin:Harwin_M20-89003xx_1x03_P2.54mm_Horizontal" (id 2) (at 41.91 73.66 0)
-      (effects (font (size 1.27 1.27)) hide)
-    )
-    (property "Datasheet" "~" (id 3) (at 41.91 73.66 0)
-      (effects (font (size 1.27 1.27)) hide)
-    )
-    (pin "1")
-    (pin "2")
-    (pin "3")
   )
   (symbol (lib_id "Device:LED") (at 52.07 59.69 90) (unit 1)
@@
       (reference "D2") (unit 1) (value "LED") (footprint "LED_SMD:LED_1210_3225Metric_Pad1.42x2.65mm_HandSolder")
     )
-    (path "/60286f78-b4bb-4f92-a0e1-bbbd3f27364c"
-      (reference "J1") (unit 1) (value "Conn_01x03_Male") (footprint "Connector_Harwin:Harwin_M20-89003xx_1x03_P2.54mm_Horizontal")
-    )
     (path "/35419037-528f-4c1c-80b4-8a6035dd7f49"
       (reference "R1") (unit 1) (value "200") (footprint "Resistor_SMD:R_1210_3225Metric_Pad1.30x2.65mm_HandSolder")
@@
       (reference "R2") (unit 1) (value "200") (footprint "Resistor_SMD:R_1210_3225Metric_Pad1.30x2.65mm_HandSolder")
     )
-  )
+    (path "/15e6f15c-c8d9-42bd-a57c-d5f9cc9ea377"
+      (reference "SW1") (unit 1) (value "SW_DPDT_x2") (footprint "MSS22D18G2:MSS22D18G2")
+    )
+    (path "/372b29d4-609a-4d2b-962b-eb70aaa3df64"
+      (reference "SW1") (unit 2) (value "SW_DPDT_x2") (footprint "MSS22D18G2:MSS22D18G2")
+    )
+  )
